Commit message: 测试了点云分割代码,obstaclelayer能显示

File: src/sentry_simulation/urdf/imu.urdf.xacro (robot description, xacro)
@@ -28,5 +28,5 @@
     </link>
     <joint name="imu_joint" type="fixed">
-        <axis xyz="0 1 0" />
+        <axis xyz="0 0 0" />
         <parent link="base_link" />
         <child link="imu_link" />
