Commit message: 修复了点云差分的bug,包括起始点不一致和时间戳的问题,添加了有移动障碍物的仿真

File: src/sentry_simulation/urdf/obstacle.urdf.xacro (robot description, xacro)
@@ -58,5 +58,5 @@
             <origin xyz="0 0 0.05" rpy="0 0 0"/>
             <geometry>
-                <box size="0.2 0.3 0.8"/>
+                <box size="0.5 0.5 0.4"/>
             </geometry>
             <material name="White" />
@@ -65,5 +65,5 @@
             <origin xyz="0 0 0.05" rpy="0 0 0"/>
             <geometry>
-                <box size="0.3 0.2 0.15"/>
+                <box size="0.5 0.5 0.4"/>
             </geometry>
         </collision>
@@ -184,12 +184,12 @@
     <xacro:gazebo_material ref="obstacle_right_rear_wheel"  color="Red" />
     <!-- //// ////////////////////////////// driver controller //////////////////////////////////  -->
-    <!-- <gazebo>
+    <gazebo>
         <plugin name="mecanum_controller" filename="libgazebo_ros_planar_move.so">
             <always_on>true</always_on>
             <updateRate>100.0</updateRate>
             <robotNamespace>/</robotNamespace>
-            <commandTopic>cmd_vel</commandTopic>
-            <odometryTopic>odom</odometryTopic>
-            <odometryFrame>odom</odometryFrame>
+            <commandTopic>obstacle/cmd_vel</commandTopic>
+            <odometryTopic>obstacle/odom</odometryTopic>
+            <odometryFrame>obstacle/odom</odometryFrame>
             <leftFrontJoint>obstacle_base_to_wheel1</leftFrontJoint>
             <rightFrontJoint>obstacle_base_to_wheel3</rightFrontJoint>
@@ -205,4 +205,4 @@
             <cmdTimeout>1.0</cmdTimeout>
         </plugin>
-    </gazebo> -->
+    </gazebo>
 </robot>
