Commit message: add relocalization pkg, fix bug in controller which set local goal repeatedly, use undistorted pointcloud to approach a better segmentation result while moving

File: src/sentry_simulation/urdf/livox_mid360.urdf.xacro (robot description, xacro)
@@ -64,6 +64,6 @@
               <samples>50</samples>
               <resolution>1</resolution>
-              <min_angle>${-7.22/180*PI}</min_angle>
-              <max_angle>${55.22/180*PI}</max_angle>
+              <min_angle>${-PI}</min_angle>
+              <max_angle>${PI}</max_angle>
             </vertical>
           </scan>

File: src/sentry_simulation/urdf/obstacle.urdf.xacro (robot description, xacro)
@@ -27,4 +27,21 @@
         </inertial>
     </xacro:macro>
+<xacro:macro name="Box_inertial_matrix" params="m l w h">
+       <inertial>
+               <mass value="${m}" />
+               <inertia ixx="${m*(h*h + l*l)/12}" ixy = "0" ixz = "0"
+                   iyy="${m*(w*w + l*l)/12}" iyz= "0"
+                   izz="${m*(w*w + h*h)/12}" />
+       </inertial>
+    </xacro:macro>
+    <!-- Defining the inertial matrix used for cylinder -->
+    <xacro:macro name="cylinder_inertial_matrix" params="m r h">
+        <inertial>
+            <mass value="${m}" />
+            <inertia ixx="${m*(3*r*r+h*h)/12}" ixy = "0" ixz = "0"
+                iyy="${m*(3*r*r+h*h)/12}" iyz = "0"
+                izz="${m*r*r/2}" />
+        </inertial>
+    </xacro:macro>
     <xacro:macro name="gazebo_material" params="ref color">
         <gazebo reference="${ref}">
@@ -68,5 +85,5 @@
             </geometry>
         </collision>
-        <xacro:inertial_matrix mass="25" />
+        <xacro:Box_inertial_matrix m="25" l="0.5" w="0.5" h="0.4"/>
     </link>
     <link name="obstacle_left_front_wheel">
@@ -84,5 +101,5 @@
             </geometry>
         </collision>
-        <xacro:inertial_matrix mass="0.5" />
+        <xacro:cylinder_inertial_matrix m="0.5" r="${radius_wheel}" h="${length_wheel}"/>
     </link>
     <link name="obstacle_right_front_wheel">
@@ -100,5 +117,5 @@
             </geometry>
         </collision>
-        <xacro:inertial_matrix mass="0.5" />
+        <xacro:cylinder_inertial_matrix m="0.5" r="${radius_wheel}" h="${length_wheel}"/>
     </link>
     <link name="obstacle_left_rear_wheel">
@@ -116,5 +133,5 @@
             </geometry>
         </collision>
-        <xacro:inertial_matrix mass="0.5" />
+        <xacro:cylinder_inertial_matrix m="0.5" r="${radius_wheel}" h="${length_wheel}"/>
     </link>
     <link name="obstacle_right_rear_wheel">
@@ -132,5 +149,5 @@
             </geometry>
         </collision>
-        <xacro:inertial_matrix mass="0.5" />
+        <xacro:cylinder_inertial_matrix m="0.5" r="${radius_wheel}" h="${length_wheel}"/>
     </link>
     <!-- //////////////////////////////// all joints ////////////////////////////////// -->

File: src/sentry_simulation/urdf/sentry_base.urdf.xacro (robot description, xacro)
@@ -27,4 +27,21 @@
         </inertial>
     </xacro:macro>
+    <xacro:macro name="Box_inertial_matrix" params="m l w h">
+       <inertial>
+               <mass value="${m}" />
+               <inertia ixx="${m*(h*h + l*l)/12}" ixy = "0" ixz = "0"
+                   iyy="${m*(w*w + l*l)/12}" iyz= "0"
+                   izz="${m*(w*w + h*h)/12}" />
+       </inertial>
+    </xacro:macro>
+    <!-- Defining the inertial matrix used for cylinder -->
+    <xacro:macro name="cylinder_inertial_matrix" params="m r h">
+        <inertial>
+            <mass value="${m}" />
+            <inertia ixx="${m*(3*r*r+h*h)/12}" ixy = "0" ixz = "0"
+                iyy="${m*(3*r*r+h*h)/12}" iyz = "0"
+                izz="${m*r*r/2}" />
+        </inertial>
+    </xacro:macro>
     <xacro:macro name="gazebo_material" params="ref color">
         <gazebo reference="${ref}">
@@ -46,8 +63,16 @@
             <origin xyz="0 0 0.05" rpy="0 0 0"/>
             <geometry>
-                <box size="0.3 0.2 0.15"/>
-            </geometry>
-        </collision>
-        <xacro:inertial_matrix mass="25" />
+                <box size="0.2 0.3 0.1"/>
+            </geometry>
+        </collision>
+        <xacro:Box_inertial_matrix m="25" l="0.2" w="0.3" h="0.1"/>
+        <!-- <inertial>
+            <mass value="25" />
+            <inertia
+            ixx="0.1" ixy="0" ixz="0"
+             iyy="0.1" iyz="0"
+             izz="0.1"
+            />
+        </inertial> -->
     </link>
     <link name="left_front_wheel">
@@ -65,5 +90,5 @@
             </geometry>
         </collision>
-        <xacro:inertial_matrix mass="0.5" />
+        <xacro:cylinder_inertial_matrix m="0.5" r="${radius_wheel}" h="${length_wheel}"/>
     </link>
     <link name="right_front_wheel">
@@ -81,5 +106,5 @@
             </geometry>
         </collision>
-        <xacro:inertial_matrix mass="0.5" />
+        <xacro:cylinder_inertial_matrix m="0.5" r="${radius_wheel}" h="${length_wheel}"/>
     </link>
     <link name="left_rear_wheel">
@@ -97,5 +122,5 @@
             </geometry>
         </collision>
-        <xacro:inertial_matrix mass="0.5" />
+        <xacro:cylinder_inertial_matrix m="0.5" r="${radius_wheel}" h="${length_wheel}"/>
     </link>
     <link name="right_rear_wheel">
@@ -113,5 +138,5 @@
             </geometry>
         </collision>
-        <xacro:inertial_matrix mass="0.5" />
+        <xacro:cylinder_inertial_matrix m="0.5" r="${radius_wheel}" h="${length_wheel}"/>
     </link>
     <!-- //////////////////////////////// all joints ////////////////////////////////// -->

Commit message: v1.0

File: src/sentry_simulation/urdf/livox_mid360.urdf.xacro (robot description, xacro)
@@ -41,5 +41,5 @@
   </link>
   <joint name="livox_mid360_joint" type="fixed">
-    <origin xyz="0 0 0.25" rpy="0 0 0" />
+    <origin xyz="0 0 0.25" rpy="-0.3491 0 0" />
     <parent link="base_link" />
     <child link="livox_mid360" />

Commit message: add custom recovery behavior, fix relocalization when drifting

File: src/sentry_simulation/urdf/livox_mid360.urdf.xacro (robot description, xacro)
@@ -41,5 +41,5 @@
   </link>
   <joint name="livox_mid360_joint" type="fixed">
-    <origin xyz="0 0 0.25" rpy="-0.3491 0 0" />
+    <origin xyz="0.189 0 0.32" rpy="0 0.3491 0" />
     <parent link="base_link" />
     <child link="livox_mid360" />
